Commit message: finish bucket and poses

File: pkg01/urdf/simple_gripper.urdf.xacro (robot description, xacro)
@@ -184,5 +184,5 @@
       <type>transmission_interface/SimpleTransmission</type>
       <joint name="${prefix}left_finger_joint">
-        <hardwareInterface>hardware_interface/EffortJointInterface</hardwareInterface>
+        <hardwareInterface>hardware_interface/PositionJointInterface</hardwareInterface>
       </joint>
       <actuator name="${prefix}left_finger_motor">
@@ -194,5 +194,5 @@
       <type>transmission_interface/SimpleTransmission</type>
       <joint name="${prefix}right_finger_joint">
-        <hardwareInterface>hardware_interface/EffortJointInterface</hardwareInterface>
+        <hardwareInterface>hardware_interface/PositionJointInterface</hardwareInterface>
       </joint>
       <actuator name="${prefix}right_finger_motor">
@@ -200,15 +200,4 @@
       </actuator>
     </transmission>
-    <!-- Gazebo Mimic Joint Plugin (makes right finger mirror left finger motion) -->
-    <gazebo>
-      <plugin name="${prefix}mimic_joint_plugin" filename="libroboticsgroup_gazebo_mimic_joint_plugin.so">
-        <joint>${prefix}left_finger_joint</joint>
-        <mimicJoint>${prefix}right_finger_joint</mimicJoint>
-        <multiplier>1.0</multiplier>
-        <offset>0.0</offset>
-        <maxEffort>100</maxEffort>
-        <robotNamespace>/</robotNamespace>
-      </plugin>
-    </gazebo>
   </xacro:macro>
 </robot>

Commit message: add new bucket collision

File: pkg01/urdf/simple_gripper.urdf.xacro (robot description, xacro)
@@ -63,5 +63,5 @@
     <link name="${prefix}left_finger">
       <visual>
-        <origin xyz="0 0 0.045" rpy="0 0 0"/>
+        <origin xyz="0 0 0.045" rpy="0 0 ${-PI/2.0}"/>
         <geometry>
           <box size="0.015 0.025 0.09"/>
@@ -70,5 +70,5 @@
       </visual>
       <collision>
-        <origin xyz="0 0 0.045" rpy="0 0 0"/>
+        <origin xyz="0 0 0.045" rpy="0 0 ${-PI/2.0}"/>
         <geometry>
           <box size="0.015 0.025 0.09"/>
@@ -76,5 +76,5 @@
       </collision>
       <inertial>
-        <origin xyz="0 0 0.045" rpy="0 0 0"/>
+        <origin xyz="0 0 0.045" rpy="0 0 ${-PI/2.0}"/>
         <mass value="0.03"/>
         <inertia ixx="0.00001" ixy="0.0" ixz="0.0"
@@ -83,8 +83,62 @@
       </inertial>
     </link>
+    <link name="${prefix}left_finger_hook">
+      <visual>
+        <origin xyz="0 -0.01 0" rpy="0 0 ${-PI/2.0}"/>
+        <geometry>
+          <box size="0.03 0.025 0.01"/>
+        </geometry>
+        <material name="${prefix}gripper_dark"/>
+      </visual>
+      <collision>
+        <origin xyz="0 -0.01 0" rpy="0 0 ${-PI/2.0}"/>
+        <geometry>
+          <box size="0.03 0.025 0.01"/>
+        </geometry>
+      </collision>
+      <inertial>
+        <origin xyz="0 -0.01 0" rpy="0 0 ${-PI/2.0}"/>
+        <mass value="0.01"/>
+        <inertia ixx="0.000005" ixy="0.0" ixz="0.0"
+                 iyy="0.000005" iyz="0.0"
+                 izz="0.000005"/>
+      </inertial>
+    </link>
+    <link name="${prefix}left_finger_hook_parallel">
+      <visual>
+        <origin xyz="0 0 -0.015" rpy="0 0 0"/>
+        <geometry>
+          <box size="0.025 0.002 0.04"/>
+        </geometry>
+        <material name="${prefix}gripper_dark"/>
+      </visual>
+      <collision>
+        <origin xyz="0 0 -0.015" rpy="0 0 0"/>
+        <geometry>
+          <box size="0.025 0.002 0.06"/>
+        </geometry>
+      </collision>
+      <inertial>
+        <origin xyz="0 0 -0.015" rpy="0 0 0"/>
+        <mass value="0.01"/>
+        <inertia ixx="0.000005" ixy="0.0" ixz="0.0"
+                 iyy="0.000005" iyz="0.0"
+                 izz="0.000005"/>
+      </inertial>
+    </link>
+    <joint name="${prefix}left_finger_hook_horizontal_joint" type="fixed">
+      <parent link="${prefix}left_finger"/>
+      <child link="${prefix}left_finger_hook"/>
+      <origin xyz="0 0 0.09" rpy="0 0 0"/>
+    </joint>
+    <joint name="${prefix}left_finger_hook_parallel_joint" type="fixed">
+      <parent link="${prefix}left_finger_hook"/>
+      <child link="${prefix}left_finger_hook_parallel"/>
+      <origin xyz="0 -0.025 0" rpy="0 0 0"/>
+    </joint>
     <!-- Right Finger -->
     <link name="${prefix}right_finger">
       <visual>
-        <origin xyz="0 0 0.045" rpy="0 0 0"/>
+        <origin xyz="0 0 0.045" rpy="0 0 ${-PI/2.0}"/>
         <geometry>
           <box size="0.015 0.025 0.09"/>
@@ -93,5 +147,5 @@
       </visual>
       <collision>
-        <origin xyz="0 0 0.045" rpy="0 0 0"/>
+        <origin xyz="0 0 0.045" rpy="0 0 ${-PI/2.0}"/>
         <geometry>
           <box size="0.015 0.025 0.09"/>
@@ -99,5 +153,5 @@
       </collision>
       <inertial>
-        <origin xyz="0 0 0.045" rpy="0 0 0"/>
+        <origin xyz="0 0 0.045" rpy="0 0 ${-PI/2.0}"/>
         <mass value="0.03"/>
         <inertia ixx="0.00001" ixy="0.0" ixz="0.0"
@@ -106,4 +160,58 @@
       </inertial>
     </link>
+    <link name="${prefix}right_finger_hook">
+      <visual>
+        <origin xyz="0 0.01 0" rpy="0 0 ${-PI/2.0}"/>
+        <geometry>
+          <box size="0.03 0.025 0.01"/>
+        </geometry>
+        <material name="${prefix}gripper_dark"/>
+      </visual>
+      <collision>
+        <origin xyz="0 0.01 0" rpy="0 0 ${-PI/2.0}"/>
+        <geometry>
+          <box size="0.03 0.025 0.01"/>
+        </geometry>
+      </collision>
+      <inertial>
+        <origin xyz="0 0.01 0" rpy="0 0 ${-PI/2.0}"/>
+        <mass value="0.01"/>
+        <inertia ixx="0.000005" ixy="0.0" ixz="0.0"
+                 iyy="0.000005" iyz="0.0"
+                 izz="0.000005"/>
+      </inertial>
+    </link>
+    <link name="${prefix}right_finger_hook_parallel">
+      <visual>
+        <origin xyz="0 0 -0.015" rpy="0 0 0"/>
+        <geometry>
+          <box size="0.025 0.002 0.04"/>
+        </geometry>
+        <material name="${prefix}gripper_dark"/>
+      </visual>
+      <collision>
+        <origin xyz="0 0 -0.015" rpy="0 0 0"/>
+        <geometry>
+          <box size="0.025 0.002 0.06"/>
+        </geometry>
+      </collision>
+      <inertial>
+        <origin xyz="0 0 -0.015" rpy="0 0 0"/>
+        <mass value="0.01"/>
+        <inertia ixx="0.000005" ixy="0.0" ixz="0.0"
+                 iyy="0.000005" iyz="0.0"
+                 izz="0.000005"/>
+      </inertial>
+    </link>
+    <joint name="${prefix}right_finger_hook_horizontal_joint" type="fixed">
+      <parent link="${prefix}right_finger"/>
+      <child link="${prefix}right_finger_hook"/>
+      <origin xyz="0 0 0.09" rpy="0 0 0"/>
+    </joint>
+    <joint name="${prefix}right_finger_hook_parallel_joint" type="fixed">
+      <parent link="${prefix}right_finger_hook"/>
+      <child link="${prefix}right_finger_hook_parallel"/>
+      <origin xyz="0 0.025 0" rpy="0 0 0"/>
+    </joint>
     <!-- Gripper Tip Link (virtual link for grasping point) -->
     <link name="${prefix}gripper_tip">
@@ -130,5 +238,5 @@
       <parent link="${prefix}gripper_palm"/>
       <child link="${prefix}left_finger"/>
-      <origin xyz="0 0.0125 0.04" rpy="0 0 0"/>
+      <origin xyz="-0.015 0.0175 0.04" rpy="0 0 0"/>
       <axis xyz="0 1 0"/>
       <limit lower="-0.0125" upper="0.025" effort="100" velocity="0.5"/>
@@ -140,5 +248,5 @@
       <parent link="${prefix}gripper_palm"/>
       <child link="${prefix}right_finger"/>
-      <origin xyz="0 -0.0125 0.04" rpy="0 0 0"/>
+      <origin xyz="0.015 -0.0175 0.04" rpy="0 0 0"/>
       <axis xyz="0 -1 0"/>
       <limit lower="-0.0125" upper="0.025" effort="100" velocity="0.5"/>
@@ -172,4 +280,40 @@
     </gazebo>
     <gazebo reference="${prefix}right_finger">
+      <material>Gazebo/DarkGrey</material>
+      <mu1>2.0</mu1>
+      <mu2>2.0</mu2>
+      <kp>1000000.0</kp>
+      <kd>100.0</kd>
+      <minDepth>0.001</minDepth>
+      <maxVel>0.1</maxVel>
+    </gazebo>
+    <gazebo reference="${prefix}left_finger_hook">
+      <material>Gazebo/DarkGrey</material>
+      <mu1>2.0</mu1>
+      <mu2>2.0</mu2>
+      <kp>1000000.0</kp>
+      <kd>100.0</kd>
+      <minDepth>0.001</minDepth>
+      <maxVel>0.1</maxVel>
+    </gazebo>
+    <gazebo reference="${prefix}right_finger_hook">
+      <material>Gazebo/DarkGrey</material>
+      <mu1>2.0</mu1>
+      <mu2>2.0</mu2>
+      <kp>1000000.0</kp>
+      <kd>100.0</kd>
+      <minDepth>0.001</minDepth>
+      <maxVel>0.1</maxVel>
+    </gazebo>
+    <gazebo reference="${prefix}left_finger_hook_parallel">
+      <material>Gazebo/DarkGrey</material>
+      <mu1>2.0</mu1>
+      <mu2>2.0</mu2>
+      <kp>1000000.0</kp>
+      <kd>100.0</kd>
+      <minDepth>0.001</minDepth>
+      <maxVel>0.1</maxVel>
+    </gazebo>
+    <gazebo reference="${prefix}right_finger_hook_parallel">
       <material>Gazebo/DarkGrey</material>
       <mu1>2.0</mu1>

Commit message: altri tentativi (NON VANNO)

File: pkg01/urdf/simple_gripper.urdf.xacro (robot description, xacro)
@@ -77,30 +77,30 @@
       <inertial>
         <origin xyz="0 0 0.045" rpy="0 0 ${-PI/2.0}"/>
-        <mass value="0.03"/>
-        <inertia ixx="0.00001" ixy="0.0" ixz="0.0"
-                 iyy="0.00001" iyz="0.0"
-                 izz="0.00001"/>
+        <mass value="0.2"/>
+        <inertia ixx="0.0001" ixy="0.0" ixz="0.0"
+                 iyy="0.0001" iyz="0.0"
+                 izz="0.0001"/>
       </inertial>
     </link>
     <link name="${prefix}left_finger_hook">
       <visual>
-        <origin xyz="0 -0.01 0" rpy="0 0 ${-PI/2.0}"/>
-        <geometry>
-          <box size="0.03 0.025 0.01"/>
-        </geometry>
-        <material name="${prefix}gripper_dark"/>
-      </visual>
-      <collision>
-        <origin xyz="0 -0.01 0" rpy="0 0 ${-PI/2.0}"/>
-        <geometry>
-          <box size="0.03 0.025 0.01"/>
-        </geometry>
-      </collision>
-      <inertial>
-        <origin xyz="0 -0.01 0" rpy="0 0 ${-PI/2.0}"/>
-        <mass value="0.01"/>
-        <inertia ixx="0.000005" ixy="0.0" ixz="0.0"
-                 iyy="0.000005" iyz="0.0"
-                 izz="0.000005"/>
+        <origin xyz="0 -0.02 0" rpy="0 0 ${-PI/2.0}"/>
+        <geometry>
+          <box size="0.05 0.025 0.01"/>
+        </geometry>
+        <material name="${prefix}gripper_dark"/>
+      </visual>
+      <collision>
+        <origin xyz="0 -0.02 0" rpy="0 0 ${-PI/2.0}"/>
+        <geometry>
+          <box size="0.05 0.025 0.01"/>
+        </geometry>
+      </collision>
+      <inertial>
+        <origin xyz="0 -0.02 0" rpy="0 0 ${-PI/2.0}"/>
+        <mass value="0.05"/>
+        <inertia ixx="0.00005" ixy="0.0" ixz="0.0"
+                 iyy="0.00005" iyz="0.0"
+                 izz="0.00005"/>
       </inertial>
     </link>
@@ -121,8 +121,8 @@
       <inertial>
         <origin xyz="0 0 -0.015" rpy="0 0 0"/>
-        <mass value="0.01"/>
-        <inertia ixx="0.000005" ixy="0.0" ixz="0.0"
-                 iyy="0.000005" iyz="0.0"
-                 izz="0.000005"/>
+        <mass value="0.05"/>
+        <inertia ixx="0.00005" ixy="0.0" ixz="0.0"
+                 iyy="0.00005" iyz="0.0"
+                 izz="0.00005"/>
       </inertial>
     </link>
@@ -135,5 +135,5 @@
       <parent link="${prefix}left_finger_hook"/>
       <child link="${prefix}left_finger_hook_parallel"/>
-      <origin xyz="0 -0.025 0" rpy="0 0 0"/>
+      <origin xyz="0 -0.045 0" rpy="0 0 0"/>
     </joint>
     <!-- Right Finger -->
@@ -154,30 +154,30 @@
       <inertial>
         <origin xyz="0 0 0.045" rpy="0 0 ${-PI/2.0}"/>
-        <mass value="0.03"/>
-        <inertia ixx="0.00001" ixy="0.0" ixz="0.0"
-                 iyy="0.00001" iyz="0.0"
-                 izz="0.00001"/>
+        <mass value="0.2"/>
+        <inertia ixx="0.0001" ixy="0.0" ixz="0.0"
+                 iyy="0.0001" iyz="0.0"
+                 izz="0.0001"/>
       </inertial>
     </link>
     <link name="${prefix}right_finger_hook">
       <visual>
-        <origin xyz="0 0.01 0" rpy="0 0 ${-PI/2.0}"/>
-        <geometry>
-          <box size="0.03 0.025 0.01"/>
-        </geometry>
-        <material name="${prefix}gripper_dark"/>
-      </visual>
-      <collision>
-        <origin xyz="0 0.01 0" rpy="0 0 ${-PI/2.0}"/>
-        <geometry>
-          <box size="0.03 0.025 0.01"/>
-        </geometry>
-      </collision>
-      <inertial>
-        <origin xyz="0 0.01 0" rpy="0 0 ${-PI/2.0}"/>
-        <mass value="0.01"/>
-        <inertia ixx="0.000005" ixy="0.0" ixz="0.0"
-                 iyy="0.000005" iyz="0.0"
-                 izz="0.000005"/>
+        <origin xyz="0 0.02 0" rpy="0 0 ${-PI/2.0}"/>
+        <geometry>
+          <box size="0.05 0.025 0.01"/>
+        </geometry>
+        <material name="${prefix}gripper_dark"/>
+      </visual>
+      <collision>
+        <origin xyz="0 0.02 0" rpy="0 0 ${-PI/2.0}"/>
+        <geometry>
+          <box size="0.05 0.025 0.01"/>
+        </geometry>
+      </collision>
+      <inertial>
+        <origin xyz="0 0.02 0" rpy="0 0 ${-PI/2.0}"/>
+        <mass value="0.05"/>
+        <inertia ixx="0.00005" ixy="0.0" ixz="0.0"
+                 iyy="0.00005" iyz="0.0"
+                 izz="0.00005"/>
       </inertial>
     </link>
@@ -198,8 +198,8 @@
       <inertial>
         <origin xyz="0 0 -0.015" rpy="0 0 0"/>
-        <mass value="0.01"/>
-        <inertia ixx="0.000005" ixy="0.0" ixz="0.0"
-                 iyy="0.000005" iyz="0.0"
-                 izz="0.000005"/>
+        <mass value="0.05"/>
+        <inertia ixx="0.00005" ixy="0.0" ixz="0.0"
+                 iyy="0.00005" iyz="0.0"
+                 izz="0.00005"/>
       </inertial>
     </link>
@@ -212,5 +212,5 @@
       <parent link="${prefix}right_finger_hook"/>
       <child link="${prefix}right_finger_hook_parallel"/>
-      <origin xyz="0 0.025 0" rpy="0 0 0"/>
+      <origin xyz="0 0.045 0" rpy="0 0 0"/>
     </joint>
     <!-- Gripper Tip Link (virtual link for grasping point) -->
@@ -234,12 +234,12 @@
     <!-- Origin at palm edge (40mm/2 = 20mm) minus finger half-width (12.5mm) = 7.5mm -->
     <!-- Lower limit (closed): fingers meet at center without overlap -->
-    <!-- Upper limit (open): 25mm travel = 50mm total grip width -->
+    <!-- Upper limit (open): 50mm travel = 100mm total grip width -->
     <joint name="${prefix}left_finger_joint" type="prismatic">
       <parent link="${prefix}gripper_palm"/>
       <child link="${prefix}left_finger"/>
-      <origin xyz="-0.015 0.0175 0.04" rpy="0 0 0"/>
+      <origin xyz="-0.015 0.0275 0.04" rpy="0 0 0"/>
       <axis xyz="0 1 0"/>
-      <limit lower="-0.0125" upper="0.025" effort="100" velocity="0.5"/>
-      <dynamics damping="1.0" friction="0.5"/>
+      <limit lower="-0.0125" upper="0.05" effort="2000" velocity="0.5"/>
+      <dynamics damping="50.0" friction="10.0"/>
     </joint>
     <!-- Joint: Right Finger (Prismatic - opens/closes) -->
@@ -248,8 +248,8 @@
       <parent link="${prefix}gripper_palm"/>
       <child link="${prefix}right_finger"/>
-      <origin xyz="0.015 -0.0175 0.04" rpy="0 0 0"/>
+      <origin xyz="0.015 -0.0275 0.04" rpy="0 0 0"/>
       <axis xyz="0 -1 0"/>
-      <limit lower="-0.0125" upper="0.025" effort="100" velocity="0.5"/>
-      <dynamics damping="1.0" friction="0.5"/>
+      <limit lower="-0.0125" upper="0.05" effort="2000" velocity="0.5"/>
+      <dynamics damping="50.0" friction="10.0"/>
     </joint>
     <!-- Joint: Palm to Gripper Tip (fixed, for reference point) -->
@@ -272,55 +272,85 @@
     <gazebo reference="${prefix}left_finger">
       <material>Gazebo/DarkGrey</material>
-      <mu1>2.0</mu1>
-      <mu2>2.0</mu2>
-      <kp>1000000.0</kp>
-      <kd>100.0</kd>
-      <minDepth>0.001</minDepth>
-      <maxVel>0.1</maxVel>
+      <mu1>3.0</mu1>
+      <mu2>3.0</mu2>
+      <kp>50000000.0</kp>
+      <kd>5000.0</kd>
+      <minDepth>0.00001</minDepth>
+      <maxVel>0.001</maxVel>
+      <fdir1>0 0 1</fdir1>
+      <softCfm>0.0</softCfm>
+      <softErp>0.9</softErp>
+      <selfCollide>true</selfCollide>
+      <gravity>false</gravity>
     </gazebo>
     <gazebo reference="${prefix}right_finger">
       <material>Gazebo/DarkGrey</material>
-      <mu1>2.0</mu1>
-      <mu2>2.0</mu2>
-      <kp>1000000.0</kp>
-      <kd>100.0</kd>
-      <minDepth>0.001</minDepth>
-      <maxVel>0.1</maxVel>
+      <mu1>3.0</mu1>
+      <mu2>3.0</mu2>
+      <kp>50000000.0</kp>
+      <kd>5000.0</kd>
+      <minDepth>0.00001</minDepth>
+      <maxVel>0.001</maxVel>
+      <fdir1>0 0 1</fdir1>
+      <softCfm>0.0</softCfm>
+      <softErp>0.9</softErp>
+      <selfCollide>true</selfCollide>
+      <gravity>false</gravity>
     </gazebo>
     <gazebo reference="${prefix}left_finger_hook">
       <material>Gazebo/DarkGrey</material>
-      <mu1>2.0</mu1>
-      <mu2>2.0</mu2>
-      <kp>1000000.0</kp>
-      <kd>100.0</kd>
-      <minDepth>0.001</minDepth>
-      <maxVel>0.1</maxVel>
+      <mu1>3.0</mu1>
+      <mu2>3.0</mu2>
+      <kp>50000000.0</kp>
+      <kd>5000.0</kd>
+      <minDepth>0.00001</minDepth>
+      <maxVel>0.001</maxVel>
+      <fdir1>0 0 1</fdir1>
+      <softCfm>0.0</softCfm>
+      <softErp>0.9</softErp>
+      <selfCollide>true</selfCollide>
+      <gravity>false</gravity>
     </gazebo>
     <gazebo reference="${prefix}right_finger_hook">
       <material>Gazebo/DarkGrey</material>
-      <mu1>2.0</mu1>
-      <mu2>2.0</mu2>
-      <kp>1000000.0</kp>
-      <kd>100.0</kd>
-      <minDepth>0.001</minDepth>
-      <maxVel>0.1</maxVel>
+      <mu1>3.0</mu1>
+      <mu2>3.0</mu2>
+      <kp>50000000.0</kp>
+      <kd>5000.0</kd>
+      <minDepth>0.00001</minDepth>
+      <maxVel>0.001</maxVel>
+      <fdir1>0 0 1</fdir1>
+      <softCfm>0.0</softCfm>
+      <softErp>0.9</softErp>
+      <selfCollide>true</selfCollide>
+      <gravity>false</gravity>
     </gazebo>
     <gazebo reference="${prefix}left_finger_hook_parallel">
       <material>Gazebo/DarkGrey</material>
-      <mu1>2.0</mu1>
-      <mu2>2.0</mu2>
-      <kp>1000000.0</kp>
-      <kd>100.0</kd>
-      <minDepth>0.001</minDepth>
-      <maxVel>0.1</maxVel>
+      <mu1>3.0</mu1>
+      <mu2>3.0</mu2>
+      <kp>50000000.0</kp>
+      <kd>5000.0</kd>
+      <minDepth>0.00001</minDepth>
+      <maxVel>0.001</maxVel>
+      <fdir1>0 0 1</fdir1>
+      <softCfm>0.0</softCfm>
+      <softErp>0.9</softErp>
+      <selfCollide>true</selfCollide>
+      <gravity>false</gravity>
     </gazebo>
     <gazebo reference="${prefix}right_finger_hook_parallel">
       <material>Gazebo/DarkGrey</material>
-      <mu1>2.0</mu1>
-      <mu2>2.0</mu2>
-      <kp>1000000.0</kp>
-      <kd>100.0</kd>
-      <minDepth>0.001</minDepth>
-      <maxVel>0.1</maxVel>
+      <mu1>3.0</mu1>
+      <mu2>3.0</mu2>
+      <kp>50000000.0</kp>
+      <kd>5000.0</kd>
+      <minDepth>0.00001</minDepth>
+      <maxVel>0.001</maxVel>
+      <fdir1>0 0 1</fdir1>
+      <softCfm>0.0</softCfm>
+      <softErp>0.9</softErp>
+      <selfCollide>true</selfCollide>
+      <gravity>false</gravity>
     </gazebo>
     <!-- Transmission for left finger (for ros_control) -->
@@ -334,4 +364,8 @@
       </actuator>
     </transmission>
+    <!-- Gazebo joint properties for left finger -->
+    <gazebo reference="${prefix}left_finger_joint">
+      <provideFeedback>true</provideFeedback>
+    </gazebo>
     <!-- Transmission for right finger (for ros_control) -->
     <transmission name="${prefix}right_finger_trans">
@@ -344,4 +378,8 @@
       </actuator>
     </transmission>
+    <!-- Gazebo joint properties for right finger -->
+    <gazebo reference="${prefix}right_finger_joint">
+      <provideFeedback>true</provideFeedback>
+    </gazebo>
   </xacro:macro>
 </robot>
