Commit message: add keypad and platform movement

File: pkg01/urdf/ur10e.urdf.xacro (robot description, xacro)
@@ -281,5 +281,5 @@
     <parent link="flange"/>
     <child link="robotiq_arg2f_base_link"/>
-    <origin xyz="0 0 0" rpy="0 0 ${PI/2}"/>
+    <origin xyz="0 0 0" rpy="0 ${PI/2} ${PI/2}"/>
   </joint>
   <!-- Gazebo plugin for ROS Control -->

Commit message: more grasp attempt

File: pkg01/urdf/ur10e.urdf.xacro (robot description, xacro)
@@ -281,6 +281,9 @@
     <parent link="flange"/>
     <child link="robotiq_arg2f_base_link"/>
-    <origin xyz="0 0 0" rpy="0 ${PI/2} ${PI/2}"/>
-  </joint>
+    <origin xyz="0 0 0" rpy="${-PI/2} 0 0"/>
+  </joint>
+  <!-- Include Gazebo properties for gripper (high friction for grasping) -->
+  <xacro:include filename="$(find pkg01)/urdf/gripper_gazebo.xacro"/>
+  <xacro:gripper_gazebo_properties prefix=""/>
   <!-- Gazebo plugin for ROS Control -->
   <gazebo>
