Commit message: add platform and bucket (wip)

File: pkg01/urdf/mobile_platform.urdf.xacro (robot description, xacro)
@@ -13,5 +13,13 @@
     </material>
     <!-- Fixed world link (ground reference) -->
-    <link name="${prefix}world_platform"/>
+    <link name="${prefix}world_platform">
+      <inertial>
+        <mass value="0.001"/>
+        <origin xyz="0 0 0" rpy="0 0 0"/>
+        <inertia ixx="0.001" ixy="0.0" ixz="0.0"
+                 iyy="0.001" iyz="0.0"
+                 izz="0.001"/>
+      </inertial>
+    </link>
     <!-- Platform base link (moves along rail) -->
     <link name="${prefix}platform_base">
@@ -79,5 +87,8 @@
       <origin xyz="0 0 ${platform_height}" rpy="0 0 0"/>
     </joint>
-    <!-- Gazebo properties for the platform -->
+    <!-- Gazebo properties -->
+    <gazebo reference="${prefix}world_platform">
+      <static>true</static>
+    </gazebo>
     <gazebo reference="${prefix}platform_base">
       <material>Gazebo/DarkGrey</material>

File: pkg01/urdf/ur10e.urdf.xacro (robot description, xacro)
@@ -263,4 +263,9 @@
     <child link="flange"/>
   </joint>
+  <!-- Include mobile platform macros -->
+  <xacro:include filename="$(find pkg01)/urdf/mobile_platform.urdf.xacro"/>
+  <!-- Instantiate the mobile platform -->
+  <xacro:mobile_platform prefix=""/>
+  <!-- Connect robot base to platform mount -->
   <joint name="robot_mount_to_base" type="fixed">
     <origin xyz="0 0 0.05" rpy="0 0 0"/>
@@ -268,12 +273,4 @@
     <child link="base_link"/>
   </joint>
-  <!-- Fix world platform link to ground in Gazebo -->
-  <gazebo reference="world_platform">
-    <static>true</static>
-  </gazebo>
-  <!-- Include mobile platform macros -->
-  <xacro:include filename="$(find pkg01)/urdf/mobile_platform.urdf.xacro"/>
-  <!-- Instantiate the mobile platform -->
-  <xacro:mobile_platform prefix=""/>
   <!-- Include gripper macros -->
  <xacro:include filename="$(find pkg01)/urdf/simple_gripper.urdf.xacro"/>

Commit message: add wheel

File: pkg01/urdf/mobile_platform.urdf.xacro (robot description, xacro)
@@ -47,4 +47,54 @@
       </inertial>
     </link>
+    <!-- Wheel properties -->
+    <xacro:property name="wheel_radius" value="0.1"/>
+    <xacro:property name="wheel_width" value="0.05"/>
+    <xacro:property name="wheel_mass" value="2.0"/>
+    <xacro:property name="wheel_offset_x" value="0.4"/>
+    <xacro:property name="wheel_offset_y" value="0.35"/>
+    <!-- Wheel macro -->
+    <xacro:macro name="platform_wheel" params="wheel_prefix x_pos y_pos">
+      <link name="${prefix}${wheel_prefix}_wheel">
+        <visual>
+          <geometry>
+            <cylinder radius="${wheel_radius}" length="${wheel_width}"/>
+          </geometry>
+          <origin xyz="0 0 0" rpy="${pi/2} 0 0"/>
+          <material name="Black">
+            <color rgba="0.1 0.1 0.1 1.0"/>
+          </material>
+        </visual>
+        <collision>
+          <geometry>
+            <cylinder radius="${wheel_radius}" length="${wheel_width}"/>
+          </geometry>
+          <origin xyz="0 0 0" rpy="${pi/2} 0 0"/>
+        </collision>
+        <inertial>
+          <mass value="${wheel_mass}"/>
+          <origin xyz="0 0 0" rpy="${pi/2} 0 0"/>
+          <inertia ixx="${(1/12) * wheel_mass * (3*wheel_radius*wheel_radius + wheel_width*wheel_width)}"
+                   ixy="0.0" ixz="0.0"
+                   iyy="${(1/12) * wheel_mass * (3*wheel_radius*wheel_radius + wheel_width*wheel_width)}"
+                   iyz="0.0"
+                   izz="${0.5 * wheel_mass * wheel_radius * wheel_radius}"/>
+        </inertial>
+      </link>
+      <joint name="${prefix}${wheel_prefix}_wheel_joint" type="fixed">
+        <parent link="${prefix}platform_base"/>
+        <child link="${prefix}${wheel_prefix}_wheel"/>
+        <origin xyz="${x_pos} ${y_pos} ${wheel_radius - platform_height/2}" rpy="0 0 0"/>
+      </joint>
+      <gazebo reference="${prefix}${wheel_prefix}_wheel">
+        <material>Gazebo/Black</material>
+        <mu1>1.0</mu1>
+        <mu2>1.0</mu2>
+      </gazebo>
+    </xacro:macro>
+    <!-- Instantiate 4 wheels -->
+    <xacro:platform_wheel wheel_prefix="front_left" x_pos="${wheel_offset_x}" y_pos="${wheel_offset_y}"/>
+    <xacro:platform_wheel wheel_prefix="front_right" x_pos="${wheel_offset_x}" y_pos="${-wheel_offset_y}"/>
+    <xacro:platform_wheel wheel_prefix="rear_left" x_pos="${-wheel_offset_x}" y_pos="${wheel_offset_y}"/>
+    <xacro:platform_wheel wheel_prefix="rear_right" x_pos="${-wheel_offset_x}" y_pos="${-wheel_offset_y}"/>
     <!-- Prismatic joint for linear motion (0 to 10 meters along X axis) -->
     <joint name="${prefix}platform_joint" type="prismatic">

Commit message: bucket fixes

File: pkg01/urdf/mobile_platform.urdf.xacro (robot description, xacro)
@@ -7,5 +7,5 @@
     <xacro:property name="platform_width" value="0.8"/>
     <xacro:property name="platform_height" value="0.15"/>
-    <xacro:property name="platform_mass" value="50.0"/>
+    <xacro:property name="platform_mass" value="500.0"/>  <!-- INCREASED from 50 to 500 kg for stability -->
     <!-- Material for platform -->
     <material name="DarkGrey">
@@ -104,5 +104,5 @@
       <axis xyz="1 0 0"/>  <!-- Motion along X axis -->
       <limit lower="0.0" upper="10.0" effort="1000.0" velocity="1.0"/>
-      <dynamics damping="50.0" friction="10.0"/>
+      <dynamics damping="500.0" friction="100.0"/>  <!-- INCREASED damping 50→500, friction 10→100 for stability -->
     </joint>
     <!-- Robot mounting plate on top of platform -->
@@ -143,6 +143,8 @@
     <gazebo reference="${prefix}platform_base">
       <material>Gazebo/DarkGrey</material>
-      <mu1>0.8</mu1>
-      <mu2>0.8</mu2>
+      <mu1>100.0</mu1>  <!-- INCREASED from 0.8 to 100 - extreme friction to prevent sliding -->
+      <mu2>100.0</mu2>  <!-- INCREASED from 0.8 to 100 - extreme friction to prevent sliding -->
+      <kp>10000000.0</kp>  <!-- Added: 10M stiffness for rigid contact -->
+      <kd>10000.0</kd>     <!-- Added: 10k damping for stability -->
     </gazebo>
     <gazebo reference="${prefix}robot_mount">
